Commit message: first commit

File: src/description/gazebo_control.xacro (robot description, xacro)
@@ -4,8 +4,12 @@
         <plugin name="gz::sim::systems::DiffDrive" filename="gz-sim-diff-drive-system">
             <!-- Wheel Information -->
-            <left_joint>left_wheel_joint</left_joint>
-            <right_joint>right_wheel_joint</right_joint>
-            <wheel_separation>0.250</wheel_separation>
-            <wheel_radius>0.05</wheel_radius>
+            <!-- <left_joint>left_wheel_joint</left_joint>
+            <right_joint>right_wheel_joint</right_joint> -->
+            <left_joint>front_left_wheel_joint</left_joint>
+            <left_joint>rear_left_wheel_joint</left_joint>
+            <right_joint>front_right_wheel_joint</right_joint>
+            <right_joint>rear_right_wheel_joint</right_joint>
+            <wheel_separation>0.297</wheel_separation>
+            <wheel_radius>0.033</wheel_radius>
             <!-- Limits -->
             <!-- <max_wheel_torque>200</max_wheel_torque> -->

File: src/description/lidar.xacro (robot description, xacro)
@@ -41,9 +41,9 @@
             <material name="red"/>
         </visual>
-        <collision>
-            <!-- <geometry>
+        <!--<collision>
+             <geometry>
                 <cylinder radius="0.05" length="0.04"/>
-            </geometry> -->
-        </collision>
+            </geometry>
+        </collision>-->
         <xacro:inertial_cylinder mass="0.1" length="0.04" radius="0.05">
             <origin xyz="0 0 0" rpy="0 0 0"/>
@@ -83,6 +83,6 @@
                     <horizontal>
                         <samples>360</samples>
-                        <min_angle>-3.14</min_angle>
-                        <max_angle>3.14</max_angle>
+                        <min_angle>-1.57</min_angle>
+                        <max_angle>1.57</max_angle>
                     </horizontal>
                 </scan>

File: src/description/robot_core.xacro (robot description, xacro)
@@ -52,5 +52,5 @@
     </link>
     <!-- LEFT WHEEL LINK -->
-    <joint name="left_wheel_joint" type="continuous">
+    <!-- <joint name="left_wheel_joint" type="continuous">
         <parent link="base_link"/>
         <child link="left_wheel"/>
@@ -73,7 +73,7 @@
             <origin xyz="0 0 0" rpy="0 0 0"/>
         </xacro:inertial_cylinder>
-    </link>
+    </link> -->
     <!-- RIGHT WHEEL LINK -->
-    <joint name="right_wheel_joint" type="continuous">
+    <!-- <joint name="right_wheel_joint" type="continuous">
         <parent link="base_link"/>
         <child link="right_wheel"/>
@@ -96,5 +96,97 @@
             <origin xyz="0 0 0" rpy="0 0 0"/>
         </xacro:inertial_cylinder>
-    </link>
+    </link> -->
+    <!-- FRONT LEFT WHEEL LINK -->
+	<joint name="front_left_wheel_joint" type="continuous">
+    	<parent link="base_link" />
+    	<child link="front_left_wheel" />
+    	<origin xyz="0.1 0.125 0" rpy="${pi/2} 0 0" />
+        <axis xyz="0 0 -1"/>
+  	</joint>
+	<link name="front_left_wheel">
+    	<visual>
+            <geometry>
+                <cylinder radius="0.05" length="0.04"/>
+            </geometry>
+            <material name="blue"/>
+        </visual>
+        <collision>
+            <geometry>
+                <cylinder radius="0.05" length="0.04"/>
+            </geometry>
+        </collision>
+        <xacro:inertial_cylinder mass="0.1" length="0.04" radius="0.05">
+            <origin xyz="0 0 0" rpy="0 0 0"/>
+        </xacro:inertial_cylinder>
+  	</link>
+    <!-- REAR LEFT WHEEL LINK -->
+	<joint name="rear_left_wheel_joint" type="continuous">
+    	<parent link="base_link" />
+    	<child link="rear_left_wheel" />
+    	<origin xyz="-0.05 0.125 0" rpy="${pi/2} 0 0" />
+        <axis xyz="0 0 -1"/>
+  	</joint>
+	<link name="rear_left_wheel">
+    	<visual>
+            <geometry>
+                <cylinder radius="0.05" length="0.04"/>
+            </geometry>
+            <material name="blue"/>
+        </visual>
+        <collision>
+            <geometry>
+                <cylinder radius="0.05" length="0.04"/>
+            </geometry>
+        </collision>
+        <xacro:inertial_cylinder mass="0.1" length="0.04" radius="0.05">
+            <origin xyz="0 0 0" rpy="0 0 0"/>
+        </xacro:inertial_cylinder>
+  	</link>
+    <!-- FRONT RIGHT WHEEL LINK -->
+	<joint name="front_right_wheel_joint" type="continuous">
+    	<parent link="base_link" />
+    	<child link="front_right_wheel" />
+    	<origin xyz="0.1 -0.125 0" rpy="${pi/2} 0 0" />
+        <axis xyz="0 0 -1"/>
+  	</joint>
+	<link name="front_right_wheel">
+    	<visual>
+            <geometry>
+                <cylinder radius="0.05" length="0.04"/>
+            </geometry>
+            <material name="blue"/>
+        </visual>
+        <collision>
+            <geometry>
+                <cylinder radius="0.05" length="0.04"/>
+            </geometry>
+        </collision>
+        <xacro:inertial_cylinder mass="0.1" length="0.04" radius="0.05">
+            <origin xyz="0 0 0" rpy="0 0 0"/>
+        </xacro:inertial_cylinder>
+  	</link>
+    <!-- REAR RIGHT WHEEL2 LINK -->
+	<joint name="rear_right_wheel_joint" type="continuous">
+    	<parent link="base_link" />
+    	<child link="rear_right_wheel" />
+    	<origin xyz="-0.05 -0.125 0" rpy="${pi/2} 0 0" />
+        <axis xyz="0 0 -1"/>
+  	</joint>
+	<link name="rear_right_wheel">
+    	<visual>
+            <geometry>
+                <cylinder radius="0.05" length="0.04"/>
+            </geometry>
+            <material name="blue"/>
+        </visual>
+        <collision>
+            <geometry>
+                <cylinder radius="0.05" length="0.04"/>
+            </geometry>
+        </collision>
+        <xacro:inertial_cylinder mass="0.1" length="0.04" radius="0.05">
+            <origin xyz="0 0 0" rpy="0 0 0"/>
+        </xacro:inertial_cylinder>
+  	</link>
     <!-- CASTER WHEEL LINK -->
     <joint name="caster_wheel_joint" type="fixed">

File: src/description/ros2_control.xacro (robot description, xacro)
@@ -11,8 +11,7 @@
                 <param name="baud_rate">57600</param>
                 <param name="timeout_ms">1000</param>
-                <!-- CHANGE ACCORDINLY -->
-                <param name="enc_counts_per_rev">200</param>
+                <param name="enc_counts_per_rev">3436</param>
             </hardware>
-            <joint name="left_wheel_joint">
+            <!-- <joint name="left_wheel_joint">
                 <command_interface name="velocity">
                     <param name="min">-10</param>
@@ -29,4 +28,36 @@
                 <state_interface name="position"/>
                 <state_interface name="velocity"/>
+            </joint> -->
+            <joint name="front_left_wheel_joint">
+                <command_interface name="velocity">
+                    <param name="min">-10</param>
+                    <param name="max">10</param>
+                </command_interface>
+                <state_interface name="position"/>
+                <state_interface name="velocity"/>
+            </joint>
+            <joint name="rear_left_wheel_joint">
+                <command_interface name="velocity">
+                    <param name="min">-10</param>
+                    <param name="max">10</param>
+                </command_interface>
+                <state_interface name="position"/>
+                <state_interface name="velocity"/>
+            </joint>
+            <joint name="front_right_wheel_joint">
+                <command_interface name="velocity">
+                    <param name="min">-10</param>
+                    <param name="max">10</param>
+                </command_interface>
+                <state_interface name="position"/>
+                <state_interface name="velocity"/>
+            </joint>
+            <joint name="rear_right_wheel_joint">
+                <command_interface name="velocity">
+                    <param name="min">-10</param>
+                    <param name="max">10</param>
+                </command_interface>
+                <state_interface name="position"/>
+                <state_interface name="velocity"/>
             </joint>
         </ros2_control>
@@ -37,5 +68,5 @@
                 <plugin>gz_ros2_control/GazeboSimSystem</plugin>
             </hardware>
-            <joint name="left_wheel_joint">
+            <!-- <joint name="left_wheel_joint">
                 <command_interface name="velocity">
                     <param name="min">-10</param>
@@ -46,4 +77,36 @@
             </joint>
             <joint name="right_wheel_joint">
+                <command_interface name="velocity">
+                    <param name="min">-10</param>
+                    <param name="max">10</param>
+                </command_interface>
+                <state_interface name="velocity"/>
+                <state_interface name="position"/>
+            </joint> -->
+            <joint name="front_left_wheel_joint">
+                <command_interface name="velocity">
+                    <param name="min">-10</param>
+                    <param name="max">10</param>
+                </command_interface>
+                <state_interface name="velocity"/>
+                <state_interface name="position"/>
+            </joint>
+            <joint name="rear_left_wheel_joint">
+                <command_interface name="velocity">
+                    <param name="min">-10</param>
+                    <param name="max">10</param>
+                </command_interface>
+                <state_interface name="velocity"/>
+                <state_interface name="position"/>
+            </joint>
+            <joint name="front_right_wheel_joint">
+                <command_interface name="velocity">
+                    <param name="min">-10</param>
+                    <param name="max">10</param>
+                </command_interface>
+                <state_interface name="velocity"/>
+                <state_interface name="position"/>
+            </joint>
+            <joint name="rear_right_wheel_joint">
                 <command_interface name="velocity">
                     <param name="min">-10</param>

Commit message: Broke some thing in gz-sim

File: src/description/gazebo_control.xacro (robot description, xacro)
@@ -11,5 +11,5 @@
             <right_joint>rear_right_wheel_joint</right_joint>
             <wheel_separation>0.297</wheel_separation>
-            <wheel_radius>0.033</wheel_radius>
+            <wheel_radius>0.05</wheel_radius>
             <!-- Limits -->
             <!-- <max_wheel_torque>200</max_wheel_torque> -->
@@ -27,6 +27,8 @@
             name="gz::sim::systems::JointStatePublisher">
             <topic>joint_states</topic>
-            <joint_name>left_wheel_joint</joint_name>
-            <joint_name>right_wheel_joint</joint_name>
+            <joint_name>front_left_wheel_joint</joint_name>
+            <joint_name>rear_left_wheel_joint</joint_name>
+            <joint_name>front_right_wheel_joint</joint_name>
+            <joint_name>rear_right_wheel_joint</joint_name>
         </plugin>
     </gazebo>

File: src/description/robot_core.xacro (robot description, xacro)
@@ -120,4 +120,9 @@
         </xacro:inertial_cylinder>
   	</link>
+    <gazebo reference="front_left_wheel">
+        <material>Gazebo/Blue</material>
+        <mu1 value="0.001"/>
+        <mu2 value="0.001"/>
+    </gazebo>
     <!-- REAR LEFT WHEEL LINK -->
 	<joint name="rear_left_wheel_joint" type="continuous">
@@ -143,4 +148,9 @@
         </xacro:inertial_cylinder>
   	</link>
+    <gazebo reference="rear_left_wheel">
+        <material>Gazebo/Blue</material>
+        <mu1 value="0.001"/>
+        <mu2 value="0.001"/>
+    </gazebo>
     <!-- FRONT RIGHT WHEEL LINK -->
 	<joint name="front_right_wheel_joint" type="continuous">
@@ -166,4 +176,9 @@
         </xacro:inertial_cylinder>
   	</link>
+    <gazebo reference="front_right_wheel">
+        <material>Gazebo/Blue</material>
+        <mu1 value="0.001"/>
+        <mu2 value="0.001"/>
+    </gazebo>
     <!-- REAR RIGHT WHEEL2 LINK -->
 	<joint name="rear_right_wheel_joint" type="continuous">
@@ -189,6 +204,11 @@
         </xacro:inertial_cylinder>
   	</link>
+    <gazebo reference="rear_right_wheel">
+        <material>Gazebo/Blue</material>
+        <mu1 value="0.001"/>
+        <mu2 value="0.001"/>
+    </gazebo>
     <!-- CASTER WHEEL LINK -->
-    <joint name="caster_wheel_joint" type="fixed">
+    <!-- <joint name="caster_wheel_joint" type="fixed">
         <parent link="chassis"/>
         <child link="caster_wheel"/>
@@ -215,4 +235,4 @@
         <mu1 value="0.001"/>
         <mu2 value="0.001"/>
-    </gazebo>
+    </gazebo> -->
 </robot>

File: src/description/ros2_control.xacro (robot description, xacro)
@@ -5,7 +5,10 @@
             <hardware>
                 <plugin>diffdrive_arduino/DiffDriveArduinoHardware</plugin>
-                <param name="left_wheel_name">left_wheel_joint</param>
-                <param name="right_wheel_name">right_wheel_joint</param>
+                <param name="front_left_wheel_name">front_left_wheel_joint</param>
+                <param name="rear_left_wheel_name">rear_left_wheel_joint</param>
+                <param name="front_right_wheel_name">front_right_wheel_joint</param>
+                <param name="rear_right_wheel_name">rear_right_wheel_joint</param>
                 <param name="loop_rate">30</param>
+                <!-- CHANGE TO THE GOOD DEVICE -->
                 <param name="device">/dev/ttyUSB0</param>
                 <param name="baud_rate">57600</param>

Commit message: Changed for nav bring up file, made the yellow path, changed map to 0 0,  fixed gz not moving

File: src/description/gazebo_control.xacro (robot description, xacro)
@@ -6,4 +6,5 @@
             <!-- <left_joint>left_wheel_joint</left_joint>
             <right_joint>right_wheel_joint</right_joint> -->
+            <num_wheel_pairs>2</num_wheel_pairs>
             <left_joint>front_left_wheel_joint</left_joint>
             <left_joint>rear_left_wheel_joint</left_joint>

File: src/description/robot_core.xacro (robot description, xacro)
@@ -120,9 +120,4 @@
         </xacro:inertial_cylinder>
   	</link>
-    <gazebo reference="front_left_wheel">
-        <material>Gazebo/Blue</material>
-        <mu1 value="0.001"/>
-        <mu2 value="0.001"/>
-    </gazebo>
     <!-- REAR LEFT WHEEL LINK -->
 	<joint name="rear_left_wheel_joint" type="continuous">
@@ -148,9 +143,4 @@
         </xacro:inertial_cylinder>
   	</link>
-    <gazebo reference="rear_left_wheel">
-        <material>Gazebo/Blue</material>
-        <mu1 value="0.001"/>
-        <mu2 value="0.001"/>
-    </gazebo>
     <!-- FRONT RIGHT WHEEL LINK -->
 	<joint name="front_right_wheel_joint" type="continuous">
@@ -176,9 +166,4 @@
         </xacro:inertial_cylinder>
   	</link>
-    <gazebo reference="front_right_wheel">
-        <material>Gazebo/Blue</material>
-        <mu1 value="0.001"/>
-        <mu2 value="0.001"/>
-    </gazebo>
     <!-- REAR RIGHT WHEEL2 LINK -->
 	<joint name="rear_right_wheel_joint" type="continuous">
@@ -204,9 +189,4 @@
         </xacro:inertial_cylinder>
   	</link>
-    <gazebo reference="rear_right_wheel">
-        <material>Gazebo/Blue</material>
-        <mu1 value="0.001"/>
-        <mu2 value="0.001"/>
-    </gazebo>
     <!-- CASTER WHEEL LINK -->
     <!-- <joint name="caster_wheel_joint" type="fixed">
