Commit message: removed top lidar, try killing, added pose for blue team

File: src/description/lidar.xacro (robot description, xacro)
@@ -1,9 +1,4 @@
 <?xml version="1.0"?>
 <robot xmlns:xacro="http://www.ros.org/wiki/xacro" >
-    <joint name="laser_joint_top" type="fixed">
-        <parent link="chassis"/>
-        <child link="laser_frame_top"/>
-        <origin xyz="0.122 0 0.212" rpy="0 0 0"/>
-    </joint>
     <joint name="laser_joint_bottom" type="fixed">
         <parent link="chassis"/>
@@ -11,27 +6,4 @@
         <origin xyz="0.35 0 0.01" rpy="0 0 0"/>
     </joint>
-    <link name="laser_frame_top">
-        <visual>
-            <geometry>
-                <cylinder radius="0.05" length="0.04"/>
-            </geometry>
-            <material name="red"/>
-        </visual>
-        <visual>
-            <origin xyz="0 0 -0.05"/>
-            <geometry>
-                <cylinder radius="0.01" length="0.1"/>
-            </geometry>
-            <material name="red"/>
-        </visual>
-        <collision>
-            <geometry>
-                <cylinder radius="0.05" length="0.04"/>
-            </geometry>
-        </collision>
-        <xacro:inertial_cylinder mass="0.1" length="0.04" radius="0.05">
-            <origin xyz="0 0 0" rpy="0 0 0"/>
-        </xacro:inertial_cylinder>
-    </link>
     <link name="laser_frame_bottom">
         <visual>
@@ -50,27 +22,4 @@
         </xacro:inertial_cylinder>
     </link>
-    <gazebo reference="laser_frame_top">
-        <material>Gazebo/Red</material>
-        <sensor name="lidar_top" type="gpu_lidar">
-            <pose> 0 0 0 0 0 0 </pose>
-            <visualize>true</visualize>
-            <update_rate>10</update_rate>
-            <lidar>
-                <scan>
-                    <horizontal>
-                        <samples>360</samples>
-                        <min_angle>-3.14</min_angle>
-                        <max_angle>3.14</max_angle>
-                    </horizontal>
-                </scan>
-                <range>
-                    <min>0.02</min>
-                    <max>12</max>
-                </range>
-            </lidar>
-            <topic>scan_top</topic>
-            <gz_frame_id>laser_frame_top</gz_frame_id>
-        </sensor>
-    </gazebo>
     <gazebo reference="laser_frame_bottom">
         <material>Gazebo/Red</material>

File: src/description/ros2_control.xacro (robot description, xacro)
@@ -1,4 +1,6 @@
 <?xml version="1.0"?>
 <robot xmlns:xacro="http://www.ros.org/wiki/xacro">
+    <!-- TODO config the values  -->
+     <!-- https://www.youtube.com/watch?v=4VVrTCnxvSw&t=342s&ab_channel=ArticulatedRobotics -->
     <xacro:unless value="$(arg sim_mode)">
         <ros2_control name="RealRobot" type="system">
