Commit message: pour ethienne et joslin !

File: src/description/robot.urdf.xacro (robot description, xacro)
@@ -12,5 +12,5 @@
     </xacro:unless>
     <xacro:include filename="lidar.xacro" />
-    <xacro:include filename="camera.xacro" />
+    <!-- <xacro:include filename="camera.xacro" /> -->
     <xacro:include filename="world.xacro" />
 </robot>

File: src/description/ros2_control.xacro (robot description, xacro)
@@ -4,34 +4,9 @@
      <!-- https://www.youtube.com/watch?v=4VVrTCnxvSw&t=342s&ab_channel=ArticulatedRobotics -->
     <xacro:unless value="$(arg sim_mode)">
-        <ros2_control name="RealRobot" type="system">
+         <ros2_control name="RealRobot" type="system">
             <hardware>
-                <plugin>diffdrive_arduino/DiffDriveArduinoHardware</plugin>
-                <param name="front_left_wheel_name">front_left_wheel_joint</param>
-                <param name="rear_left_wheel_name">rear_left_wheel_joint</param>
-                <param name="front_right_wheel_name">front_right_wheel_joint</param>
-                <param name="rear_right_wheel_name">rear_right_wheel_joint</param>
-                <param name="loop_rate">30</param>
-                <!-- CHANGE TO THE GOOD DEVICE -->
-                <param name="device">/dev/ttyUSB0</param>
-                <param name="baud_rate">57600</param>
-                <param name="timeout_ms">1000</param>
-                <param name="enc_counts_per_rev">3436</param>
+                <!-- use a generic hardware interface; odom is computed by your diff_drive controller -->
+                <plugin>mock_components/GenericSystem</plugin>
             </hardware>
-            <!-- <joint name="left_wheel_joint">
-                <command_interface name="velocity">
-                    <param name="min">-10</param>
-                    <param name="max">10</param>
-                </command_interface>
-                <state_interface name="position"/>
-                <state_interface name="velocity"/>
-            </joint>
-            <joint name="right_wheel_joint">
-                <command_interface name="velocity">
-                    <param name="min">-10</param>
-                    <param name="max">10</param>
-                </command_interface>
-                <state_interface name="position"/>
-                <state_interface name="velocity"/>
-            </joint> -->
             <joint name="front_left_wheel_joint">
                 <command_interface name="velocity">
@@ -73,20 +48,4 @@
                 <plugin>gz_ros2_control/GazeboSimSystem</plugin>
             </hardware>
-            <!-- <joint name="left_wheel_joint">
-                <command_interface name="velocity">
-                    <param name="min">-10</param>
-                    <param name="max">10</param>
-                </command_interface>
-                <state_interface name="velocity"/>
-                <state_interface name="position"/>
-            </joint>
-            <joint name="right_wheel_joint">
-                <command_interface name="velocity">
-                    <param name="min">-10</param>
-                    <param name="max">10</param>
-                </command_interface>
-                <state_interface name="velocity"/>
-                <state_interface name="position"/>
-            </joint> -->
             <joint name="front_left_wheel_joint">
                 <command_interface name="velocity">
